Commit message: added depth camera and lidar gazebo links

File: adiona_ws/adiona_pkg/models/adiona.urdf (robot description, URDF)
Before this commit: robot adiona, 8 links, 7 joints
Links:
- added link camera_depth_frame
- added link camera_link, mass 0.035; collision box size=0.015 0.130 0.022; visual box size=0.015 0.10 0.022
Joints:
- added joint camera_depth_joint: type fixed, parent camera_link, child camera_depth_frame, origin xyz=0 0 0 rpy=${-pi/2} 0 ${-pi/2}
- added joint camera_joint: type fixed, parent base_link, child camera_link, origin xyz=.01 -.025 0.04 rpy=0 0 0

Commit message: fixed urdf

File: adiona_ws/adiona_pkg/models/adiona.urdf (robot description, URDF)
Before this commit: robot adiona, 10 links, 9 joints
Links:
- added link gps_link
Joints:
- added joint gps_joint: type fixed, parent base_link, child gps_link, origin xyz=-.1 -.025 0.06 rpy=0 0 0
